File: zc-detector.kicad_sch (KiCad schematic)
At the start: 13 parts, among them Q1 MMBT2222ALT1G, U1 VOL617A

Commit message: Added some test points. Added RS-485 Module. Updated PBC.
Parts:
- added TP6: TestPointZC, TestPoint:TestPoint_THTPad_D2.0mm_Drill1.0mm, symbol Connector:TestPoint
Connections:
- net at R6.2, U1.1: now also TP6.1
Changed lines of the file:
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@@
   (junction (at 113.03 104.14) (diameter 0) (color 0 0 0 0)
   )
+  (junction (at 168.91 95.25) (diameter 0) (color 0 0 0 0)
+  )
   (junction (at 146.05 95.25) (diameter 0) (color 0 0 0 0)
   )
@@
   )
   (wire (pts (xy 99.06 104.14) (xy 101.6 104.14))
+    (stroke (width 0) (type default))
+  )
+  (wire (pts (xy 168.91 90.17) (xy 168.91 95.25))
     (stroke (width 0) (type default))
   )
@@
         )
       )
+    )
+  )
+  (symbol (lib_id "Connector:TestPoint") (at 168.91 90.17 0) (unit 1)
+    (in_bom yes) (on_board yes) (dnp no) (fields_autoplaced)
+    (property "Reference" "TP6" (at 171.45 86.233 0)
+      (effects (font (size 1.27 1.27)) (justify left))
+    )
+    (property "Value" "TestPointZC" (at 171.45 88.773 0)
+      (effects (font (size 1.27 1.27)) (justify left))
+    )
+    (property "Footprint" "TestPoint:TestPoint_THTPad_D2.0mm_Drill1.0mm" (at 173.99 90.17 0)
+      (effects (font (size 1.27 1.27)) hide)
+    )
+    (property "Datasheet" "~" (at 173.99 90.17 0)
+      (effects (font (size 1.27 1.27)) hide)
+    )
+    (pin "1")
+    (instances
+      (project "Rev1"
+        (path "/71908919-2b0a-47a6-84be-12fefaa6e518"
+          (reference "TP6") (unit 1)
+        )
+        (path "/71908919-2b0a-47a6-84be-12fefaa6e518/5081f111-7078-43b0-82cf-1fe66b064440"
+          (reference "TP7") (unit 1)
+        )
+      )
